Commit message: Pose camera: ribbon end away from the scan window
The Pi NoIR v2 was drawn with its ribbon connector toward the wrist, so
its ribbon had to run back over the scan window. Turn it 180 deg about its
lens axis, as it is fitted on the rig. Its holes are symmetric, so the
housing's standoffs don't move (housing.stl is unchanged) and the lens
sits on the other hole row, 12.28 mm further from the window
(z_pose = z_mirror + 34.28).

The URDF's pose_camera_joint now carries the full turn: the export writes
roll, pitch and yaw, and the xacro uses all three. Head CoM moves 0.2 mm.
A description test checks the connector end faces away from the window.
The manual and cad/README say which way round to fit it.

Co-Authored-By: Claude Opus 5.5 (1M context) <noreply@anthropic.com>
Claude-Session: https://claude.ai/code/session_01VvGKDo8vRKNBrUtyUKeJ5L

File: ros2/so101_scan_description/urdf/scan_head.xacro (robot description, xacro)
@@ -67,5 +67,5 @@
       <xacro:property name="folded_rpy" value="${2 * mirror_rest + pi} 0 0"/>
       <xacro:property name="pose_camera_xyz" value="${pose_camera_x} ${pose_camera_y} ${pose_camera_z}"/>
-      <xacro:property name="pose_camera_rpy" value="${pose_camera_roll} 0 0"/>
+      <xacro:property name="pose_camera_rpy" value="${pose_camera_roll} ${pose_camera_pitch} ${pose_camera_yaw}"/>
       <xacro:property name="line_half_length" value="${scan_line_half_length}"/>
     </xacro:if>

File: ros2/so101_scan_description/urdf/scan_head_params.xacro (robot description, xacro)
@@ -36,7 +36,9 @@
   <xacro:property name="pose_camera_x" value="0"/>
   <xacro:property name="pose_camera_y" value="0.02172"/>
-  <xacro:property name="pose_camera_z" value="0.05112"/>
-  <!-- board frame: +Z out of the lens, +Y toward the wrist -->
-  <xacro:property name="pose_camera_roll" value="-1.570796"/>
+  <xacro:property name="pose_camera_z" value="0.0634"/>
+  <!-- board frame: +Z out of the lens, +Y toward its ribbon connector (away from the wrist), +X along the head's -X -->
+  <xacro:property name="pose_camera_roll" value="1.570796"/>
+  <xacro:property name="pose_camera_pitch" value="0"/>
+  <xacro:property name="pose_camera_yaw" value="-3.141593"/>
   <!-- PCB back to the front of the lens module (RPI-CAM-V2 drawing) -->
   <xacro:property name="pose_camera_lens" value="0.0045"/>
@@ -46,5 +48,5 @@
   <xacro:property name="head_com_x" value="-0.0106"/>
   <xacro:property name="head_com_y" value="-0.0012"/>
-  <xacro:property name="head_com_z" value="0.0559"/>
+  <xacro:property name="head_com_z" value="0.0561"/>
   <!-- inertia of a solid box the head's size (64 x 53 x 136 mm) about the centre of mass -->
   <xacro:property name="head_ixx" value="0.000333"/>
