Commit message: Refit the URDF's head to the Edmund mirror, filter and field lens
Re-exported from main's CAD with export_head_from_cad.py: the objective
sits at 50.12 mm, the mirror station at 29.12 mm, and the head weighs
188.2 g with its centre of mass at (-10.6, -1.1, 55.5) mm. The line camera
check now takes its expected position from cad/build_report.json instead of
hard-coded numbers, and the shipped plans are regenerated for the new head
(their joints move by up to 0.7 deg).

File: ros2/so101_scan_description/urdf/scan_head_params.xacro (robot description, xacro)
@@ -10,5 +10,5 @@
   <xacro:property name="head_mount_z" value="-0.003"/>
   <!-- scan mirror shaft axis (along X), Y (y_shaft) -->
-  <xacro:property name="mirror_shaft_y" value="-0.002313"/>
+  <xacro:property name="mirror_shaft_y" value="-0.0023"/>
   <!-- scan mirror shaft axis, Z (z_shaft) -->
   <xacro:property name="mirror_shaft_z" value="0.0241"/>
@@ -16,5 +16,5 @@
   <xacro:property name="mirror_rest" value="0.785398"/>
   <!-- mirror front surface to the shaft axis (mirror_e) -->
-  <xacro:property name="mirror_face_offset" value="0.0061"/>
+  <xacro:property name="mirror_face_offset" value="0.0071"/>
   <!-- mirror angle where the hall sensor sees the magnet (mirror_home, -40 deg) -->
   <xacro:property name="mirror_home" value="-0.698132"/>
@@ -22,7 +22,7 @@
   <xacro:property name="mirror_scan_half" value="0.10472"/>
   <!-- optical axis Y (y_axis) -->
-  <xacro:property name="objective_y" value="0.002"/>
+  <xacro:property name="objective_y" value="0.00272"/>
   <!-- objective principal plane Z (z_obj) -->
-  <xacro:property name="objective_z" value="0.049413"/>
+  <xacro:property name="objective_z" value="0.05012"/>
   <!-- objective to the in-focus scan line, along the folded axis (scene_dist) -->
   <xacro:property name="scene_distance" value="0.15"/>
@@ -35,6 +35,6 @@
   <!-- Pi NoIR v2 pose camera board, lens centre on the PCB back -->
   <xacro:property name="pose_camera_x" value="0"/>
-  <xacro:property name="pose_camera_y" value="0.021"/>
-  <xacro:property name="pose_camera_z" value="0.050413"/>
+  <xacro:property name="pose_camera_y" value="0.02172"/>
+  <xacro:property name="pose_camera_z" value="0.05112"/>
   <!-- board frame: +Z out of the lens, +Y toward the wrist -->
   <xacro:property name="pose_camera_roll" value="-1.570796"/>
@@ -42,12 +42,12 @@
   <xacro:property name="pose_camera_lens" value="0.0045"/>
   <!-- mass budget in cad/build_report.json, wrist puck included -->
-  <xacro:property name="head_mass" value="0.1875"/>
+  <xacro:property name="head_mass" value="0.1882"/>
   <!-- centre of mass in the head frame (build_report.json) -->
-  <xacro:property name="head_com_x" value="-0.0107"/>
-  <xacro:property name="head_com_y" value="-0.0014"/>
-  <xacro:property name="head_com_z" value="0.0552"/>
-  <!-- inertia of a solid box the head's size (66 x 53 x 134 mm) about the centre of mass -->
-  <xacro:property name="head_ixx" value="0.000326"/>
-  <xacro:property name="head_iyy" value="0.000351"/>
-  <xacro:property name="head_izz" value="0.000112"/>
+  <xacro:property name="head_com_x" value="-0.0106"/>
+  <xacro:property name="head_com_y" value="-0.0011"/>
+  <xacro:property name="head_com_z" value="0.0555"/>
+  <!-- inertia of a solid box the head's size (66 x 53 x 135 mm) about the centre of mass -->
+  <xacro:property name="head_ixx" value="0.000331"/>
+  <xacro:property name="head_iyy" value="0.000355"/>
+  <xacro:property name="head_izz" value="0.000113"/>
 </robot>

Commit message: Re-export the ROS 2 scan head from the refitted CAD

File: ros2/so101_scan_description/urdf/scan_head_params.xacro (robot description, xacro)
@@ -42,12 +42,12 @@
   <xacro:property name="pose_camera_lens" value="0.0045"/>
   <!-- mass budget in cad/build_report.json, wrist puck included -->
-  <xacro:property name="head_mass" value="0.1882"/>
+  <xacro:property name="head_mass" value="0.1847"/>
   <!-- centre of mass in the head frame (build_report.json) -->
-  <xacro:property name="head_com_x" value="-0.0106"/>
-  <xacro:property name="head_com_y" value="-0.0011"/>
-  <xacro:property name="head_com_z" value="0.0555"/>
+  <xacro:property name="head_com_x" value="-0.0108"/>
+  <xacro:property name="head_com_y" value="-0.0012"/>
+  <xacro:property name="head_com_z" value="0.0554"/>
   <!-- inertia of a solid box the head's size (66 x 53 x 135 mm) about the centre of mass -->
-  <xacro:property name="head_ixx" value="0.000331"/>
-  <xacro:property name="head_iyy" value="0.000355"/>
-  <xacro:property name="head_izz" value="0.000113"/>
+  <xacro:property name="head_ixx" value="0.000324"/>
+  <xacro:property name="head_iyy" value="0.000349"/>
+  <xacro:property name="head_izz" value="0.00011"/>
 </robot>

Commit message: Cut the clamp's magnet pocket for the 5 x 1.6 mm magnets
The pocket was 0.4 mm too deep for the magnets on hand, which left the
magnet's face 1.5 mm from the A3144 instead of 1.1 mm. mag_t is now 1.6
mm (measured), so the pocket depth follows it. Only mirror_clamp.stl
changes; the build report and the ROS 2 head export are refreshed.

File: ros2/so101_scan_description/urdf/scan_head_params.xacro (robot description, xacro)
@@ -42,5 +42,5 @@
   <xacro:property name="pose_camera_lens" value="0.0045"/>
   <!-- mass budget in cad/build_report.json, wrist puck included -->
-  <xacro:property name="head_mass" value="0.1847"/>
+  <xacro:property name="head_mass" value="0.1846"/>
   <!-- centre of mass in the head frame (build_report.json) -->
   <xacro:property name="head_com_x" value="-0.0108"/>
@@ -49,5 +49,5 @@
   <!-- inertia of a solid box the head's size (66 x 53 x 135 mm) about the centre of mass -->
   <xacro:property name="head_ixx" value="0.000324"/>
-  <xacro:property name="head_iyy" value="0.000349"/>
+  <xacro:property name="head_iyy" value="0.000348"/>
   <xacro:property name="head_izz" value="0.00011"/>
 </robot>

Commit message: Add the controller tray and the hall breakout to the CAD
The KiCad boards in pcb/ now have a place in the model. A printed tray
holds the scan-mirror controller on the table behind the SO-101's base,
on four posts with M3 heat-set inserts, with two table-screw slots that
find a hole on a 1 in or 25 mm grid. The hall breakout lies on the
head's +X face over the A3144's lead slot, and a 0.8 mm recess in the
housing behind its lower half takes the solder on the back of its cable
pads and the strain-relief thread between its tie holes.

The breakout's M2 hole is left unused: the wall behind it is 2.5 mm
with the mirror clamp turning 1 mm inside it.

New Params cells for both boards (tagged pcb) and the tray. The model,
STLs, STEP, build report and the ROS 2 head export are rebuilt; only
housing.stl changes among the existing STLs, and controller_tray.stl
is new.

File: ros2/so101_scan_description/urdf/scan_head_params.xacro (robot description, xacro)
@@ -42,12 +42,12 @@
   <xacro:property name="pose_camera_lens" value="0.0045"/>
   <!-- mass budget in cad/build_report.json, wrist puck included -->
-  <xacro:property name="head_mass" value="0.1846"/>
+  <xacro:property name="head_mass" value="0.1851"/>
   <!-- centre of mass in the head frame (build_report.json) -->
   <xacro:property name="head_com_x" value="-0.0108"/>
   <xacro:property name="head_com_y" value="-0.0012"/>
-  <xacro:property name="head_com_z" value="0.0554"/>
-  <!-- inertia of a solid box the head's size (66 x 53 x 135 mm) about the centre of mass -->
-  <xacro:property name="head_ixx" value="0.000324"/>
-  <xacro:property name="head_iyy" value="0.000348"/>
-  <xacro:property name="head_izz" value="0.00011"/>
+  <xacro:property name="head_com_z" value="0.0553"/>
+  <!-- inertia of a solid box the head's size (64 x 53 x 135 mm) about the centre of mass -->
+  <xacro:property name="head_ixx" value="0.000325"/>
+  <xacro:property name="head_iyy" value="0.000346"/>
+  <xacro:property name="head_izz" value="0.000108"/>
 </robot>

Commit message: Fit the head to the bought optics (layout E) and screw on the hall breakout
The head now holds the optics where layout E of optics/spectrograph_model.py
puts them:

- params.py reads layout E. The field lens sits curved side toward the slit,
  flat face on a ledge in the slit block, and the collimator moves 1.76 mm
  back, to 26.76 mm behind the slit, where the slit's image through the
  thick lens is (field_dz). The grating, camera lens and board move back
  with it, so the head is 1.26 mm longer.
- The 1.2 mm stop plate at the front of the filter cap becomes a 0.6 mm
  washer with a 4 mm hole on the objective's front face, with the long-pass
  disc in front of it. A 5 mm washer is printed too, to compare at first
  light.
- The objective is the CIL161's listed 15.6 mm.

The hall breakout's M2 hole moved in pcb/ (#41) to where an M2 x 5 clears
the mirror clamp, so the board is screwed on rather than glued. The board
model's hole and screw follow it, the +X wall gets the pilot, and the mirror
sweep checks the screw tip (1.3 mm, about 1 mm to the thread).

optics_check.py compares the as-built spacings with layout E using the
model's traced numbers (4.1 nm, as in E). The calibration kit's design map
keeps config C's ideal thin lenses but takes the bought objective's 15.6 mm
and f/3.9, so the simulator's objective matches the URDF's again, and sim's
objective test takes the new numbers. Layout E's real field lens would also
stretch the slit's image unevenly along its length, by up to about 12 px,
which hsical's rows don't model, so the map leaves it out. The drift
check's test bounded a knocked instrument's tilts at 0.15 nm, which is the
plane fit's own noise on the synthetic frames (0.12 to 0.17 nm over seeds,
with the old map or the new); it now uses the check's 0.2 nm limit.

The ROS 2 head is re-exported. Two arm-safety tests that pinned the
stretched-out arm's load at 74% now allow for the mass budget moving (75%
now).

File: ros2/so101_scan_description/urdf/scan_head_params.xacro (robot description, xacro)
@@ -28,7 +28,7 @@
   <xacro:property name="scene_distance" value="0.15"/>
   <!-- half length of the scan line on the scene (half_line) -->
-  <xacro:property name="scan_line_half_length" value="0.020937"/>
+  <xacro:property name="scan_line_half_length" value="0.021538"/>
   <!-- objective focal length (f_obj) -->
-  <xacro:property name="objective_focal_length" value="0.016"/>
+  <xacro:property name="objective_focal_length" value="0.0156"/>
   <!-- slit length (slit_len) -->
   <xacro:property name="slit_length" value="0.005"/>
@@ -42,12 +42,12 @@
   <xacro:property name="pose_camera_lens" value="0.0045"/>
   <!-- mass budget in cad/build_report.json, wrist puck included -->
-  <xacro:property name="head_mass" value="0.1851"/>
+  <xacro:property name="head_mass" value="0.1868"/>
   <!-- centre of mass in the head frame (build_report.json) -->
-  <xacro:property name="head_com_x" value="-0.0108"/>
+  <xacro:property name="head_com_x" value="-0.0107"/>
   <xacro:property name="head_com_y" value="-0.0012"/>
-  <xacro:property name="head_com_z" value="0.0553"/>
-  <!-- inertia of a solid box the head's size (64 x 53 x 135 mm) about the centre of mass -->
-  <xacro:property name="head_ixx" value="0.000325"/>
-  <xacro:property name="head_iyy" value="0.000346"/>
+  <xacro:property name="head_com_z" value="0.0559"/>
+  <!-- inertia of a solid box the head's size (64 x 53 x 136 mm) about the centre of mass -->
+  <xacro:property name="head_ixx" value="0.000334"/>
+  <xacro:property name="head_iyy" value="0.000355"/>
   <xacro:property name="head_izz" value="0.000108"/>
 </robot>
