Commit message: Open up the lid's pocket for the stepper's pilot boss
The 8HS11's boss measures 16.0 mm, not the 15.0 estimate, and the pocket
drawn at 15.5 mm printed at about 15.3. Set mot_boss_d to the measured
16.0 and size the pocket with a new boss_clear param of 0.4 mm per side,
so it is drawn at 16.8 and prints near 16.6: about 0.3 mm a side on the
boss. The screw and bolt holes are unchanged.

Rebuilt with FreeCAD 1.1.3: lid.stl is the only STL that changed. Also
regenerated the STEP, .FCStd, build report and the URDF head params
(lid 0.1 g lighter).

Co-Authored-By: Claude Opus 5.5 (1M context) <noreply@anthropic.com>
Claude-Session: https://claude.ai/code/session_01JmDgATv9khuDqQP3UMnL2P

File: ros2/so101_scan_description/urdf/scan_head_params.xacro (robot description, xacro)
@@ -42,12 +42,12 @@
   <xacro:property name="pose_camera_lens" value="0.0045"/>
   <!-- mass budget in cad/build_report.json, wrist puck included -->
-  <xacro:property name="head_mass" value="0.1868"/>
+  <xacro:property name="head_mass" value="0.1867"/>
   <!-- centre of mass in the head frame (build_report.json) -->
-  <xacro:property name="head_com_x" value="-0.0107"/>
+  <xacro:property name="head_com_x" value="-0.0106"/>
   <xacro:property name="head_com_y" value="-0.0012"/>
   <xacro:property name="head_com_z" value="0.0559"/>
   <!-- inertia of a solid box the head's size (64 x 53 x 136 mm) about the centre of mass -->
-  <xacro:property name="head_ixx" value="0.000334"/>
-  <xacro:property name="head_iyy" value="0.000355"/>
+  <xacro:property name="head_ixx" value="0.000333"/>
+  <xacro:property name="head_iyy" value="0.000354"/>
   <xacro:property name="head_izz" value="0.000108"/>
 </robot>
