File: pcb/scan_controller/scan_controller.kicad_pcb (KiCad board)
At the start: 2 copper layers, 95 x 66 mm, 26 parts, among them J1 12V 5.5x2.1, J2 12V, J3 NEMA 8, J4 A3144, J5 Jetson, U1 ESP32-DevKitC (38-pin), U2 BTT TMC2209 V1.3

Commit message: Add a status LED to the controller and correct the PCB notes
A review of the merged boards against the real parts found:

- The firmware's status LED on GPIO 2 doesn't exist on a genuine
  ESP32-DevKitC, so the controller now has one: D4 (red) through R8
  (1 k) to GND, which also keeps the strapping pin low at boot.
- The 12 V terminal's + and - marks sat under its plastic body; they
  are now beside it.
- The A3144's leads leave the bottom of its body, so they run below
  the head wall's current lead slot. The README now gives the hall
  board's position for leads bent under the body and the CAD change
  the slot needs.
- README: exclude WROVER DevKitCs (GPIO 16/17 are their PSRAM), give
  the TMC2209 V1.3's pin labels, fix the regulator rationale, the
  terminal height, J5's direction, the tie holes (thread, not cable
  ties), JLCPCB's default HASL, and the library and rebuild notes.
Parts:
- added D4: red, rig:LED_0805_2012Metric, F.Cu at (104.2, 117.8)
- added R8: 1k, rig:R_0805_2012Metric, F.Cu at (108.2, 117.8)
Connections:
- U1 pad 34: unconnected-(U1-IO2-Pad34) -> /STATUS
Routing:
- net /STATUS: track 0.00 -> 4.81 mm
- net /STATUS_LED: track 0.00 -> 2.20 mm
- net GND: track 9.66 -> 11.0 mm, vias 14 -> 15
Other:
- board text added: "STATUS"
